File: pcb/digiMatex_DS410.kicad_pcb (KiCad board)
At the start: 2 copper layers, 180 x 115 mm, 37 parts, among them J1 POWER, J2 E, J3 A/B, J4 Buttons, Q1 PN2222A, Q2 PN2222A, Q3 PN2222A, U1 MAX7219

Commit message: final pcb layout
Parts:
- removed A1: mini-360, pl_dcdc:mini-360
- removed R10, R8, R9: 10k, Resistor_THT:R_Axial_DIN0207_L6.3mm_D2.5mm_P15.24mm_Horizontal
- added C3: 0.33u, Capacitor_THT:CP_Radial_D6.3mm_P2.50mm, F.Cu at (60.0, 80.6)
- added C4: 0.1u, Capacitor_THT:CP_Radial_D6.3mm_P2.50mm, F.Cu at (60.0, 95.7)
- added HS1: Heatsink, pl_heatsink:TO-220hs_16x16x25mm_2pins, F.Cu at (71.2, 88.2)
- added U2: L7805, Package_TO_SOT_THT:TO-220-3_Vertical, F.Cu at (64.7, 85.7)
- U1: moved to B.Cu
- moved R2 312.7 mm to (217.8, 97.8), turned to 180 degrees
- moved R3 290.8 mm to (210.3, 109.7), turned to 180 degrees
- moved A3 282.0 mm to (197.5, 44.8)
- moved Q1 239.2 mm to (212.9, 105.1), turned to 180 degrees
- moved JP2 170.7 mm to (149.4, 49.1), turned to 90 degrees
- moved R7 169.0 mm to (210.3, 120.0), turned to 180 degrees
- moved R6 166.1 mm to (219.9, 129.9), turned to 180 degrees
- moved JP1 162.0 mm to (165.9, 49.1), turned to -90 degrees
- moved Q2 156.6 mm to (216.9, 126.3)
- moved U1 149.5 mm to (70.1, 120.0), turned to -90 degrees
- moved R5 148.1 mm to (217.8, 101.3), turned to 180 degrees
- moved A2 147.4 mm to (170.9, 68.9), turned to -90 degrees
- moved Q3 142.4 mm to (212.8, 115.0), turned to 180 degrees
- moved C2 142.2 mm to (56.2, 117.6), turned to -90 degrees
- moved R1 137.3 mm to (60.0, 105.2), turned to -90 degrees
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Connections:
- A3 pad 12: /b_display -> unconnected-(A3-Pad12)
- A3 pad 13: /b_unit -> unconnected-(A3-Pad13)
- A3 pad 15: /b_tare -> unconnected-(A3-Pad15)
- A3 pad 23: unconnected-(A3-Pad23) -> /b_tare
- A3 pad 24: unconnected-(A3-Pad24) -> /b_unit
- A3 pad 26: unconnected-(A3-Pad26) -> /b_display
- A3 pad 7: /DT -> /SCK
- A3 pad 8: /SCK -> /DT
- J4 pad 3: /b_tare -> /b_unit
- J4 pad 5: /b_unit -> /b_tare
Routing:
- net +5V: track 0.00 -> 336.1 mm
- net /G: track 0.00 -> 230.5 mm
- net /6: track 0.00 -> 223.6 mm
- net /F: track 0.00 -> 220.5 mm
- net /MOSI: track 0.00 -> 213.4 mm
- net /4: track 0.00 -> 202.0 mm
- net /CLK: track 0.00 -> 197.4 mm, vias 0 -> 2
- net /CS: track 0.00 -> 183.7 mm, vias 0 -> 2
- net /2: track 0.00 -> 177.7 mm, vias 0 -> 2
- net /0: track 0.00 -> 160.5 mm
- net /B: track 0.00 -> 137.8 mm, vias 0 -> 2
- net /C: track 0.00 -> 135.9 mm
- net /E: track 0.00 -> 134.7 mm
- net /DP: track 0.00 -> 133.6 mm
- net /A: track 0.00 -> 131.7 mm
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- added copper zone on B.Cu, net +5V
- added copper zone on B.Cu, net GND
- added copper zone on B.Cu, net Net-(C1-Pad1)
Other:
- outline, holes or cut-outs redrawn
