File: pcb/digiMatex_DS410.kicad_pcb (KiCad board)
At the start: 2 copper layers, 180 x 115 mm, 37 parts, among them J1 POWER, J2 E, J3 A/B, J4 Buttons, Q1 PN2222A, Q2 PN2222A, Q3 PN2222A, U1 MAX7219, U2 L7805

Commit message: start pcb layout rev A
Parts:
- removed A3: ESP32-DevKitC-V4, pl_esp:esp32_devkitc_v4
- removed JP1: B-/A-, Connector_PinHeader_2.54mm:PinHeader_1x03_P2.54mm_Vertical
- removed JP2: B+/A+, Connector_PinHeader_2.54mm:PinHeader_1x03_P2.54mm_Vertical
- added C10: 10u, Capacitor_THT:CP_Radial_D6.3mm_P2.50mm, F.Cu at (150.6, 8.81)
- added C5: 100n, Capacitor_SMD:C_0603_1608Metric, F.Cu at (143.4, 18.9)
- added C6: 22u, Capacitor_SMD:C_1206_3216Metric, F.Cu at (129.4, 27.2)
- added C7: 100n, Capacitor_SMD:C_0603_1608Metric, F.Cu at (143.4, 21.4)
- added C8: 100n, Capacitor_SMD:C_0603_1608Metric, F.Cu at (151.4, 19.5)
- added C9: 10u, Capacitor_THT:CP_Radial_D6.3mm_P2.50mm, F.Cu at (136.2, 23.6)
- added J5: SCALE, TerminalBlock_Phoenix:TerminalBlock_Phoenix_MKDS-1,5-6_1x06_P5.00mm_Horizontal, B.Cu at (225.0, 87.0)
- added R10: 4k7, Capacitor_SMD:C_0603_1608Metric, F.Cu at (147.4, 18.9)
- added R11: 0, Capacitor_SMD:C_0805_2012Metric, F.Cu at (143.6, 16.1)
- added R12: 0, Capacitor_SMD:C_0805_2012Metric, F.Cu at (150.1, 14.2)
- added R13: 0, Capacitor_SMD:C_0805_2012Metric, F.Cu at (133.7, 30.4)
- added R8: 10k, Capacitor_SMD:C_0603_1608Metric, F.Cu at (151.4, 17.0)
- added R9: 4k7, Capacitor_SMD:C_0603_1608Metric, F.Cu at (147.4, 21.4)
- added SW1: SW_Push, Button_Switch_THT:SW_PUSH_6mm, F.Cu at (167.5, -4.95)
- added SW2: SW_Push, Button_Switch_THT:SW_PUSH_6mm, F.Cu at (118.0, 27.6)
- added U3: ESP32-WROOM-32E, RF_Module:ESP32-WROOM-32, B.Cu at (187.5, 53.2)
- added U4: NCP1117DT33G, Package_TO_SOT_SMD:TO-252-2, F.Cu at (110.0, 29.6)
- A2, C1, C3, C4, D1, HS1, J1, J4: moved to B.Cu
- C2: value 0.1u -> 100n; footprint Capacitor_THT:C_Disc_D4.3mm_W1.9mm_P5.00mm -> Capacitor_SMD:C_0603_1608Metric
- J2: value E -> JTAG; footprint pl_TerminalBlock:WJ127-5.0-2P -> Connector_PinHeader_2.54mm:PinHeader_2x05_P2.54mm_Vertical
- J3: value A/B -> PROG; footprint pl_TerminalBlock:WJ127-5.0-2P -> Connector_PinHeader_2.54mm:PinHeader_2x03_P2.54mm_Vertical
- Q1, Q2, Q3: value PN2222A -> MMBT3904; footprint Package_TO_SOT_THT:TO-92_Inline -> Package_TO_SOT_SMD:SOT-23
- R1, R2, R4, R5: footprint Resistor_THT:R_Axial_DIN0207_L6.3mm_D2.5mm_P15.24mm_Horizontal -> Capacitor_SMD:C_0603_1608Metric
- R3, R6, R7: value 330 -> 470; footprint Resistor_THT:R_Axial_DIN0207_L6.3mm_D2.5mm_P15.24mm_Horizontal -> Capacitor_SMD:C_0805_2012Metric
- U2: value L7805 -> L7805CDT-TR; moved to B.Cu
- moved R6 223.0 mm to (58.1, -23.5), turned to 0 degrees
- moved R7 212.5 mm to (53.7, -23.5), turned to 0 degrees
- moved R3 203.7 mm to (53.7, -20.5), turned to 0 degrees
- moved R5 199.6 mm to (62.4, -23.8), turned to 0 degrees
- moved R2 199.5 mm to (53.5, -15.3), turned to 0 degrees
- moved R4 195.6 mm to (57.5, -17.8), turned to 0 degrees
- moved C2 135.4 mm to (53.5, -17.8), turned to 0 degrees
- moved Q2 132.8 mm to (158.2, 7.11)
- moved R1 126.1 mm to (57.9, -20.8), turned to 0 degrees
- moved Q3 118.5 mm to (129.0, 31.1), turned to 0 degrees
- moved Q1 110.9 mm to (167.9, 3.80), turned to 0 degrees
- moved A2 107.2 mm to (278.1, 64.3)
- moved J2 49.5 mm to (135.8, 7.21), turned to 0 degrees
- moved J3 39.2 mm to (142.9, 7.21), turned to 0 degrees
- moved C4 14.1 mm to (74.0, 96.2), turned to 0 degrees
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Connections:
- A2 pad 8: /SCK -> /SCALE_SCK
- A2 pad 9: /DT -> /SCALE_DT
- J2 pad 1: /E+ -> +3V3
- J2 pad 2: /E- -> /ESP_TMS
- J3 pad 1: Net-(J3-Pad1) -> /EN
- Q1 pad 1: GND -> Net-(Q1-Pad1)
- Q1 pad 2: Net-(Q1-Pad2) -> GND
- Q2 pad 1: GND -> Net-(Q2-Pad1)
- Q2 pad 2: Net-(Q2-Pad2) -> GND
- Q3 pad 1: GND -> Net-(Q3-Pad1)
- Q3 pad 2: Net-(Q3-Pad2) -> GND
- R2 pad 1: Net-(Q1-Pad2) -> Net-(Q2-Pad1)
- R3 pad 1: Net-(Q1-Pad3) -> Net-(Q2-Pad3)
- R4 pad 1: Net-(Q2-Pad2) -> Net-(Q1-Pad1)
- R5 pad 1: Net-(Q3-Pad2) -> Net-(Q3-Pad1)
- R6 pad 1: Net-(Q2-Pad3) -> Net-(Q1-Pad3)
- U1 pad 1: /MOSI -> /7SEG_MOSI
- U1 pad 12: /CS -> /7SEG_CS
- U1 pad 13: /CLK -> /7SEG_CLK
Routing:
- net /MOSI: track 213.4 -> 0.00 mm
- net /CLK: track 197.4 -> 0.00 mm, vias 2 -> 0
- net /CS: track 183.7 -> 0.00 mm, vias 2 -> 0
- net +5V: track 336.1 -> 211.3 mm
- net /b_tare: track 58.0 -> 0.00 mm
- net /b_unit: track 54.8 -> 0.00 mm
- net +3V3: track 52.8 -> 0.00 mm
- net /b_display: track 52.6 -> 0.00 mm
- net /kg_LED: track 45.2 -> 0.00 mm
- net /lbs_LED: track 44.3 -> 0.00 mm
- net /WiFi_LED: track 43.3 -> 0.00 mm
- net /SCK: track 38.7 -> 0.00 mm
- net /DT: track 35.8 -> 0.00 mm
- net Net-(Q2-Pad2): track 35.7 -> 0.00 mm
- net /7SEG_CLK: track 0.00 -> 27.7 mm, vias 0 -> 2
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Other:
- outline, holes or cut-outs redrawn

Commit message: rev A layout
Parts:
- removed HS1: Heatsink, pl_heatsink:TO-220hs_16x16x25mm_2pins
- added G***: LOGO, pl_logo:logo_height_20mm, F.Cu at (88.7, 84.0)
- added G***: LOGO, pl_logo:logo_height_20mm, B.Cu at (119.9, 90.0)
- C10, C2, C5, C6, C7, C8, C9, J2, J3, Q1, Q2, Q3, SW1, SW2, U4: moved to B.Cu
- R1, R10, R2, R4, R5, R8, R9: footprint Capacitor_SMD:C_0603_1608Metric -> Resistor_SMD:R_0603_1608Metric_Pad0.98x0.95mm_HandSolder; moved to B.Cu
- R11, R12, R13: footprint Capacitor_SMD:C_0805_2012Metric -> Resistor_SMD:R_0805_2012Metric_Pad1.20x1.40mm_HandSolder; moved to B.Cu
- R3, R6, R7: footprint Capacitor_SMD:C_0805_2012Metric -> Resistor_THT:R_Axial_DIN0207_L6.3mm_D2.5mm_P10.16mm_Horizontal; moved to B.Cu
- U2: footprint Package_TO_SOT_THT:TO-220-3_Vertical -> Package_TO_SOT_SMD:TO-252-2
- moved R6 164.1 mm to (172.8, 93.8), turned to -90 degrees
- moved R3 160.8 mm to (166.8, 93.8), turned to -90 degrees
- moved R7 158.9 mm to (160.7, 93.8), turned to -90 degrees
- moved R4 153.9 mm to (171.8, 85.2), turned to 90 degrees
- moved R2 150.7 mm to (165.8, 85.2), turned to 90 degrees
- moved R1 149.0 mm to (70.2, 127.7)
- moved R5 146.2 mm to (159.8, 85.2), turned to 90 degrees
- moved C2 140.4 mm to (59.6, 122.5)
- moved D7 119.7 mm to (85.0, 120.0)
- moved J2 99.2 mm to (213.4, 68.9), turned to 180 degrees
- moved Q1 86.1 mm to (172.8, 89.8), turned to -90 degrees
- moved SW1 83.7 mm to (184.8, 76.9)
- moved Q2 83.1 mm to (166.8, 89.8), turned to -90 degrees
- moved A2 81.9 mm to (199.3, 87.0), turned to 180 degrees
- moved C6 76.3 mm to (202.9, 47.7), turned to -90 degrees
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Connections:
- U3 pad 31: /b_unit -> /b_display
- U3 pad 33: /b_display -> /b_unit
Routing:
- net +3V3: track 0.00 -> 201.4 mm, vias 0 -> 44
- net /7SEG_MOSI: track 0.00 -> 168.8 mm
- net /b_tare: track 0.00 -> 150.3 mm
- net /b_unit: track 0.00 -> 144.6 mm
- net /b_display: track 0.00 -> 139.5 mm
- net /7SEG_CS: track 16.0 -> 154.6 mm, vias 2 -> 4
- net /7SEG_CLK: track 27.7 -> 165.5 mm, vias 2 -> 4
- net Net-(D7-Pad1): track 0.00 -> 103.7 mm, vias 0 -> 1
- net +5V: track 211.3 -> 292.0 mm
- net /EN: track 0.00 -> 73.1 mm, vias 0 -> 2
- net /kg_LED: track 0.00 -> 64.8 mm
- net /lbs_LED: track 0.00 -> 60.8 mm
- net /WiFi_LED: track 0.00 -> 56.8 mm
- net /SCALE_SCK: track 0.00 -> 54.0 mm
- net /SCALE_DT: track 0.00 -> 49.2 mm
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- added copper zone on B.Cu, net +3V3
- added copper zone on F.Cu, net +3V3
- added copper zone on F.Cu, net GND
Other:
- board text added: "3V3"
- board text added: "A+"
- board text added: "A-"
- board text added: "B+"
- board text added: "B-"
- board text added: "Back Door"
- board text added: "Center Button"
- board text added: "DigiMatex DS410 Replacement Board"
- board text added: "E+"
- board text added: "E-"
- board text added: "February 2022"
- board text added: "GND"
- board text added: "IO0"
- board text added: "JTAG"
- board text added: "Left Button"
- board text added: "PROG"
- board text added: "Program"
- board text added: "RESET"
- board text added: "RXD0"
- board text added: "Reset"
- board text added: "Right Button"
- board text added: "Sam Perry"
- board text added: "TCK"
- board text added: "TDI"
- board text added: "TDO"
- board text added: "TMS"
- board text added: "TXD0"
- board text added: "github.com/sdp8483/DigiMatex_DS410_repair"

Commit message: rev b layout
Parts:
- added C11: 100n, Capacitor_SMD:C_0603_1608Metric, B.Cu at (201.3, 87.5)
- added C12: 100n, Capacitor_SMD:C_0603_1608Metric, B.Cu at (192.8, 89.3)
- added C13: 10u, Capacitor_SMD:C_0805_2012Metric_Pad1.18x1.45mm_HandSolder, B.Cu at (200.9, 90.3)
- added C14: 100n, Capacitor_SMD:C_0603_1608Metric, B.Cu at (205.8, 100.0)
- added C15: 100n, Capacitor_SMD:C_0603_1608Metric, B.Cu at (206.1, 84.1)
- added C16: 10u, Capacitor_SMD:C_0805_2012Metric_Pad1.18x1.45mm_HandSolder, B.Cu at (205.8, 86.3)
- added C17: 100n, Capacitor_SMD:C_0603_1608Metric, B.Cu at (201.3, 104.2)
- added C18: 100n, Capacitor_SMD:C_0603_1608Metric, B.Cu at (201.3, 106.2)
- added L1: 4.7uH, Inductor_SMD:L_0805_2012Metric_Pad1.05x1.20mm_HandSolder, B.Cu at (205.8, 93.2)
- added NT1: NetTie_2, NetTie:NetTie-2_SMD_Pad2.0mm, F.Cu at (199.1, 97.8)
- added Q4: PMBT2907A,215, Package_TO_SOT_SMD:SOT-23, B.Cu at (205.8, 89.5)
- added R14: 10k, Resistor_SMD:R_0603_1608Metric_Pad0.98x0.95mm_HandSolder, B.Cu at (192.6, 91.3)
- added R15: 0, Resistor_SMD:R_0603_1608Metric_Pad0.98x0.95mm_HandSolder, B.Cu at (192.6, 93.3)
- added R16: 20k, Resistor_SMD:R_0805_2012Metric_Pad1.20x1.40mm_HandSolder, B.Cu at (205.8, 95.5)
- added R17: 8.2k, Resistor_SMD:R_0805_2012Metric_Pad1.20x1.40mm_HandSolder, B.Cu at (205.8, 97.8)
- added R18: 100, Resistor_SMD:R_0603_1608Metric_Pad0.98x0.95mm_HandSolder, B.Cu at (205.8, 104.2)
- added R19: 100, Resistor_SMD:R_0603_1608Metric_Pad0.98x0.95mm_HandSolder, B.Cu at (205.8, 102.0)
- added R20: 100, Resistor_SMD:R_0603_1608Metric_Pad0.98x0.95mm_HandSolder, B.Cu at (205.8, 108.2)
- added R21: 100, Resistor_SMD:R_0603_1608Metric_Pad0.98x0.95mm_HandSolder, B.Cu at (205.8, 106.2)
- added U5: HX711, Package_SO:SOP-16_3.9x9.9mm_P1.27mm, B.Cu at (199.1, 97.8)
- turned R13 to 180 degrees
Connections:
- net /A+ renamed /Load Cell Amplifier with ADC/A+
- net /A- renamed /Load Cell Amplifier with ADC/A-
- net /B+ renamed /Load Cell Amplifier with ADC/B+
- net /B- renamed /Load Cell Amplifier with ADC/B-
- net /E+ renamed /Load Cell Amplifier with ADC/E+
- net /E- renamed GNDA
- A2 pad 8: /SCALE_SCK -> /Load Cell Amplifier with ADC/SCK
- A2 pad 9: /SCALE_DT -> /Load Cell Amplifier with ADC/DT
- R13 pad 1: Net-(J3-Pad2) -> +3V3
- R13 pad 2: +3V3 -> Net-(J3-Pad2)
- U3 pad 8: /SCALE_SCK -> /Load Cell Amplifier with ADC/DT
- U3 pad 9: /SCALE_DT -> /Load Cell Amplifier with ADC/SCK
Routing:
- net /Load Cell Amplifier with ADC/SCK: track 0.00 -> 68.0 mm
- net /Load Cell Amplifier with ADC/DT: track 0.00 -> 65.4 mm, vias 0 -> 1
- net /SCALE_SCK: track 54.0 -> 0.00 mm
- net /SCALE_DT: track 49.2 -> 0.00 mm
- net +5V: track 292.0 -> 334.0 mm, vias 0 -> 1
- net +3V3: track 201.4 -> 223.0 mm, vias 44 -> 45
- net Net-(C18-Pad1): track 0.00 -> 17.5 mm
- net /Load Cell Amplifier with ADC/B-: track 17.1 -> 33.3 mm
- net /Load Cell Amplifier with ADC/B+: track 18.8 -> 34.5 mm
- net /Load Cell Amplifier with ADC/E+: track 13.0 -> 28.0 mm
- net /Load Cell Amplifier with ADC/A+: track 16.0 -> 31.0 mm
- net Net-(C18-Pad2): track 0.00 -> 14.8 mm
- net /Load Cell Amplifier with ADC/A-: track 15.0 -> 29.2 mm
- net Net-(L1-Pad2): track 0.00 -> 12.1 mm
- net GNDA: track 14.0 -> 1.92 mm, vias 0 -> 57
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- added copper zone on B.Cu, net GNDA
- added copper zone on F.Cu, net GNDA
