File: pcb/digiMatex_DS410.kicad_sch (KiCad schematic)
At the start: 49 parts, among them J1 POWER, J2 JTAG, J3 PROG, J4 Buttons, J5 SCALE, Q1 MMBT3904, Q2 MMBT3904, Q3 MMBT3904, SW1 SW_Push, SW2 SW_Push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

Commit message: rev b layout
Connections:
- net Load Cell Amplifier with ADC/DT: now also U3.8 (IO32); no longer U3.9 (IO33)
- net Load Cell Amplifier with ADC/SCK: now also U3.9 (IO33); no longer U3.8 (IO32)
Changed lines of the file:
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@@
       (effects (font (size 1.27 1.27)) (justify left top))
     )
-    (pin "SCK" input (at 81.28 132.08 180)
+    (pin "SCK" input (at 81.28 134.62 180)
       (effects (font (size 1.27 1.27)) (justify left))
     )
-    (pin "DT" input (at 81.28 134.62 180)
+    (pin "DT" input (at 81.28 132.08 180)
       (effects (font (size 1.27 1.27)) (justify left))
     )
@@
     )
     (path "/b15ac447-b464-4fdc-8fab-1e76e308caef/a5cfd453-563e-4a0c-a405-86a4a4eaaaf9"
-      (reference "C13") (unit 1) (value "10u") (footprint "Capacitor_SMD:C_1210_3225Metric_Pad1.33x2.70mm_HandSolder")
+      (reference "C13") (unit 1) (value "10u") (footprint "Capacitor_SMD:C_0805_2012Metric_Pad1.18x1.45mm_HandSolder")
     )
     (path "/b15ac447-b464-4fdc-8fab-1e76e308caef/2863324e-f952-45aa-9849-9bd1c78b3969"
@@
     )
     (path "/b15ac447-b464-4fdc-8fab-1e76e308caef/d2655d0a-ba89-4028-b480-9460e909a178"
-      (reference "C16") (unit 1) (value "10u") (footprint "Capacitor_SMD:C_1210_3225Metric_Pad1.33x2.70mm_HandSolder")
+      (reference "C16") (unit 1) (value "10u") (footprint "Capacitor_SMD:C_0805_2012Metric_Pad1.18x1.45mm_HandSolder")
     )
     (path "/b15ac447-b464-4fdc-8fab-1e76e308caef/24b4d1bb-1df9-45fb-b154-5b56a30b369e"

Commit message: add load cell pinout
Other:
- note added: "Load Cell Pinout Ext+ -> RED Ext- -> WHT A- -> YLW A+ -> GRN"
Changed lines of the file:
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@@
     (comment 1 "PCB to be maufactured by prototype board house (JLCPCB)")
   )
+  (bus_alias "Buttons" (members "b_display" "b_tare" "b_unit"))
+  (bus_alias "HX711" (members "SCK" "DT"))
+  (bus_alias "MAX7219" (members "CLK" "MOSI" "CS"))
+  (bus_alias "LED" (members "WiFi_LED" "lbs_LED" "kg_LED"))
   (bus_alias "7Seg" (members "A" "B" "C" "D" "E" "F" "G" "DP" "1" "2" "3" "4" "5" "6" "7" "0"))
-  (bus_alias "LED" (members "WiFi_LED" "lbs_LED" "kg_LED"))
-  (bus_alias "MAX7219" (members "CLK" "MOSI" "CS"))
-  (bus_alias "HX711" (members "SCK" "DT"))
-  (bus_alias "Buttons" (members "b_display" "b_tare" "b_unit"))
   (junction (at 110.49 34.29) (diameter 0) (color 0 0 0 0)
   )
@@
     (effects (font (size 1.27 1.27)) (justify left bottom))
   )
+  (text "Load Cell Pinout\nExt+ -> RED\nExt- -> WHT\nA-	 -> YLW\nA+   -> GRN"
+    (at 128.27 139.7 0)
+    (effects (font (size 1.27 1.27)) (justify left bottom))
+  )
